File: _autosave-keyboard.sch (KiCad schematic (older format))
At the start: 68 parts, among them M1 `, M10 9, M11 0, M12 -, M13 =, M14 Backspace, M15 Tab, M16 Q, M17 W, M18 E, M19 R, M2 1, M20 T, M21 Y, M22 U, M23 I, M24 O, M25 P, M26 [, M27 ], M28 \\, M29 CapsLock, M3 2, M30 A, M31 S, M32 D, M33 F, M34 G, M35 H, M36 J, M37 K, M38 L, M39 ;, M4 3, M40 ', M41 Enter, M42 LeftShift, M43 Z, M44 X, M45 C, M46 V, M47 B, M48 N, M49 M, M5 4, M50 ,, M51 ., M52 /, M53 RightShift, M54 LeftCtrl, M55 LeftSuper, M56 LeftAlt, M57 SpaceBar, M58 RightAlt, M59 RightSuper, M6 5, M60 Menu, M61 RightCtrl, M7 6, M8 7, M9 8, U1 ROW_1_2, U2 ROW_3_4, U3 ROW_5_6, U3 SeeeduinoXIAO, U4 ROW_7_8

Commit message: Reworked layout, everything is aligned now.
Parts:
- renumbered U3 to C1
Changed lines of the file:
@@
 $EndComp
 $Comp
-L RP2040:SeeeduinoXIAO U3
+L RP2040:SeeeduinoXIAO C1
 U 1 1 617DF93D
 P 5450 1450
-F 0 "U3" H 5425 511 50  0000 C CNN
+F 0 "C1" H 5425 511 50  0000 C CNN
 F 1 "SeeeduinoXIAO" H 5425 420 50  0000 C CNN
 F 2 "RP2040:Seeeduino XIAO-MOUDLE14P-2.54-21X17.8MM" H 5100 1650 50  0001 C CNN
