File: _autosave-keyboard.sch (KiCad schematic (older format))
At the start: 54 parts, among them M1 Tab, M10 O, M11 P, M12 Backspace, M13 Esc, M14 A, M15 S, M16 D, M17 F, M18 G, M19 H, M2 Q, M20 J, M21 K, M22 L, M23 ;, M24 ', M25 Shift, M26 Z, M27 X, M28 C, M29 V, M3 W, M30 B, M31 N, M32 M, M33 ,, M34 ., M35 /, M36 Enter, M37 Blnk, M38 Ctrl, M39 Alt, M4 E, M40 Super, M41 Down, M42 Space, M43 Up, M44 L_Ar, M45 D_Ar, M46 U_Ar, M47 R_Ar, M5 R, M6 T, M7 Y, M8 U, M9 I, U1 ROW_1, U2 ROW_2, U3 ROW_3, U4 ROW_4

Commit message: Prototype 1
Parts:
- added H1, H2, H3, H4, H? (x2): MountingHole, MountingHole:MountingHole_3.2mm_M3_Pad, symbol Mechanical:MountingHole
Changed lines of the file:
@@
 	0    -1   -1   0
 $EndComp
+$Comp
+L Mechanical:MountingHole H2
+U 1 1 62183D28
+P 6950 2150
+F 0 "H2" H 7050 2196 50  0000 L CNN
+F 1 "MountingHole" H 7050 2105 50  0000 L CNN
+F 2 "MountingHole:MountingHole_3.2mm_M3_Pad" H 6950 2150 50  0001 C CNN
+F 3 "~" H 6950 2150 50  0001 C CNN
+	1    6950 2150
+	1    0    0    -1
+$EndComp
+$Comp
+L Mechanical:MountingHole H1
+U 1 1 62184586
+P 6950 1950
+F 0 "H1" H 7050 1996 50  0000 L CNN
+F 1 "MountingHole" H 7050 1905 50  0000 L CNN
+F 2 "MountingHole:MountingHole_3.2mm_M3_Pad" H 6950 1950 50  0001 C CNN
+F 3 "~" H 6950 1950 50  0001 C CNN
+	1    6950 1950
+	1    0    0    -1
+$EndComp
+$Comp
+L Mechanical:MountingHole H3
+U 1 1 62184C5C
+P 6950 2350
+F 0 "H3" H 7050 2396 50  0000 L CNN
+F 1 "MountingHole" H 7050 2305 50  0000 L CNN
+F 2 "MountingHole:MountingHole_3.2mm_M3_Pad" H 6950 2350 50  0001 C CNN
+F 3 "~" H 6950 2350 50  0001 C CNN
+	1    6950 2350
+	1    0    0    -1
+$EndComp
+$Comp
+L Mechanical:MountingHole H4
+U 1 1 6218533F
+P 6950 2550
+F 0 "H4" H 7050 2596 50  0000 L CNN
+F 1 "MountingHole" H 7050 2505 50  0000 L CNN
+F 2 "MountingHole:MountingHole_3.2mm_M3_Pad" H 6950 2550 50  0001 C CNN
+F 3 "~" H 6950 2550 50  0001 C CNN
+	1    6950 2550
+	1    0    0    -1
+$EndComp
+$Comp
+L Mechanical:MountingHole H?
+U 1 1 621C9116
+P 6950 2750
+F 0 "H?" H 7050 2796 50  0000 L CNN
+F 1 "MountingHole" H 7050 2705 50  0000 L CNN
+F 2 "MountingHole:MountingHole_3.2mm_M3_Pad" H 6950 2750 50  0001 C CNN
+F 3 "~" H 6950 2750 50  0001 C CNN
+	1    6950 2750
+	1    0    0    -1
+$EndComp
+$Comp
+L Mechanical:MountingHole H?
+U 1 1 621C92B7
+P 6950 2950
+F 0 "H?" H 7050 2996 50  0000 L CNN
+F 1 "MountingHole" H 7050 2905 50  0000 L CNN
+F 2 "MountingHole:MountingHole_3.2mm_M3_Pad" H 6950 2950 50  0001 C CNN
+F 3 "~" H 6950 2950 50  0001 C CNN
+	1    6950 2950
+	1    0    0    -1
+$EndComp
 $EndSCHEMATC
