File: keyboard.kicad_pcb (KiCad board)
At the start: 2 copper layers, 129 parts, among them M1 SWITCH-SPST-2TV, M10 SWITCH-SPST-2TV, M11 SWITCH-SPST-2TV, M12 SWITCH-SPST-2TV, M13 SWITCH-SPST-2TV, M14 SWITCH-SPST-2TV, M15 SWITCH-SPST-2TV, M16 SWITCH-SPST-2TV, M17 SWITCH-SPST-2TV, M18 SWITCH-SPST-2TV, M19 SWITCH-SPST-2TV, M2 SWITCH-SPST-2TV, M20 SWITCH-SPST-2TV, M21 SWITCH-SPST-2TV, M22 SWITCH-SPST-2TV, M23 SWITCH-SPST-2TV, M24 SWITCH-SPST-2TV, M25 SWITCH-SPST-2TV, M26 SWITCH-SPST-2TV, M27 SWITCH-SPST-2TV, M28 SWITCH-SPST-2TV, M29 SWITCH-SPST-2TV, M3 SWITCH-SPST-2TV, M30 SWITCH-SPST-2TV, M31 SWITCH-SPST-2TV, M32 SWITCH-SPST-2TV, M33 SWITCH-SPST-2TV, M34 SWITCH-SPST-2TV, M35 SWITCH-SPST-2TV, M36 SWITCH-SPST-2TV, M37 SWITCH-SPST-2TV, M38 SWITCH-SPST-2TV, M39 SWITCH-SPST-2TV, M4 SWITCH-SPST-2TV, M40 SWITCH-SPST-2TV, M41 SWITCH-SPST-2TV, M42 SWITCH-SPST-2TV, M43 SWITCH-SPST-2TV, M44 SWITCH-SPST-2TV, M45 SWITCH-SPST-2TV, M46 SWITCH-SPST-2TV, M47 SWITCH-SPST-2TV, M48 SWITCH-SPST-2TV, M49 SWITCH-SPST-2TV, M5 SWITCH-SPST-2TV, M50 SWITCH-SPST-2TV, M51 SWITCH-SPST-2TV, M52 SWITCH-SPST-2TV, M53 SWITCH-SPST-2TV, M54 SWITCH-SPST-2TV, M55 SWITCH-SPST-2TV, M56 SWITCH-SPST-2TV, M57 SWITCH-SPST-2TV, M58 SWITCH-SPST-2TV, M59 SWITCH-SPST-2TV, M6 SWITCH-SPST-2TV, M60 SWITCH-SPST-2TV, M61 SWITCH-SPST-2TV, M7 SWITCH-SPST-2TV, M8 SWITCH-SPST-2TV, M9 SWITCH-SPST-2TV, U1 PCF8575TS_1,118, U2 PCF8575TS_1,118, U3 SeeeduinoXIAO, U4 PCF8575TS_1,118, U5 PCF8575TS_1,118

Commit message: small revision
Parts:
- moved U3 250.1 mm to (46.0, 38.1)
- moved U1 241.7 mm to (294.5, 31.0)
- moved U5 235.4 mm to (294.5, 65.9)
- moved U2 130.7 mm to (24.6, 49.2)
- moved U4 111.4 mm to (24.6, 83.3)

Commit message: Reworked layout, everything is aligned now.
Parts:
- removed R10, R11, R12, R13, R14, R15, R16, R17, R18, R19, R20, R21, R22, R23, R24, R25, R26, R27, R28, R29, R3, R30, R31, R32, R33, R34, R35, R36, R37, R38, R39, R4, R40, R41, R42, R43, R44, R45, R46, R47, R48, R49, R5, R50, R51, R52, R53, R54, R55, R56, R57, R58, R59, R6, R60, R61, R62, R63, R7, R8, R9: R_Small, Resistor_SMD:R_0603_1608Metric
- removed U5: PCF8575TS_1,118, NXP:NXP-SOT340-1-02_2016-0-MFG
- added C1: SeeeduinoXIAO, RP2040:Seeeduino XIAO-MOUDLE14P-2.54-21X17.8MM, F.Cu at (-13.5, 66.7)
- M1: value SWITCH-SPST-2TV -> `; footprint Kailh_Pog:SW_Kailh_Choc_V1_2.00u -> Kailh_Pog:SW_Kailh_Choc_V1_1.00u
- M10: value SWITCH-SPST-2TV -> 9; footprint Kailh_Pog:SW_Kailh_Choc_V1_1.25u -> Kailh_Pog:SW_Kailh_Choc_V1_1.00u
- M11: value SWITCH-SPST-2TV -> 0; footprint Kailh_Pog:SW_Kailh_Choc_V1_1.25u -> Kailh_Pog:SW_Kailh_Choc_V1_1.00u
- M12: value SWITCH-SPST-2TV -> -; footprint Kailh_Pog:SW_Kailh_Choc_V1_1.25u -> Kailh_Pog:SW_Kailh_Choc_V1_1.00u
- M13: value SWITCH-SPST-2TV -> =; footprint Kailh_Pog:SW_Kailh_Choc_V1_1.25u -> Kailh_Pog:SW_Kailh_Choc_V1_1.00u
- M14: value SWITCH-SPST-2TV -> Backspace; footprint Kailh_Pog:SW_Kailh_Choc_V1_1.25u -> Kailh_Pog:SW_Kailh_Choc_V1_2.00u
- M15: value SWITCH-SPST-2TV -> Tab; footprint Kailh_Pog:SW_Kailh_Choc_V1_6.25u -> Kailh_Pog:SW_Kailh_Choc_V1_1.50u
- M16: value SWITCH-SPST-2TV -> Q
- M17: value SWITCH-SPST-2TV -> W
- M18: value SWITCH-SPST-2TV -> E
- M19: value SWITCH-SPST-2TV -> R
- M2: value SWITCH-SPST-2TV -> 1; footprint Kailh_Pog:SW_Kailh_Choc_V1_1.50u -> Kailh_Pog:SW_Kailh_Choc_V1_1.00u
- M20: value SWITCH-SPST-2TV -> T
- M21: value SWITCH-SPST-2TV -> Y
- M22: value SWITCH-SPST-2TV -> U
- M23: value SWITCH-SPST-2TV -> I
- M24: value SWITCH-SPST-2TV -> O
- M25: value SWITCH-SPST-2TV -> P
- M26: value SWITCH-SPST-2TV -> [
- M27: value SWITCH-SPST-2TV -> ]
- M28: value SWITCH-SPST-2TV -> \; footprint Kailh_Pog:SW_Kailh_Choc_V1_1.00u -> Kailh_Pog:SW_Kailh_Choc_V1_1.50u
- M29: value SWITCH-SPST-2TV -> CapsLock; footprint Kailh_Pog:SW_Kailh_Choc_V1_1.00u -> Kailh_Pog:SW_Kailh_Choc_V1_1.75u
- M3: value SWITCH-SPST-2TV -> 2; footprint Kailh_Pog:SW_Kailh_Choc_V1_1.50u -> Kailh_Pog:SW_Kailh_Choc_V1_1.00u
- M30: value SWITCH-SPST-2TV -> A
- M31: value SWITCH-SPST-2TV -> S
- M32: value SWITCH-SPST-2TV -> D
- M33: value SWITCH-SPST-2TV -> F
- M34: value SWITCH-SPST-2TV -> G
- M35: value SWITCH-SPST-2TV -> H
- M36: value SWITCH-SPST-2TV -> J
- M37: value SWITCH-SPST-2TV -> K
- M38: value SWITCH-SPST-2TV -> L
- M39: value SWITCH-SPST-2TV -> ;
- M4: value SWITCH-SPST-2TV -> 3; footprint Kailh_Pog:SW_Kailh_Choc_V1_1.75u -> Kailh_Pog:SW_Kailh_Choc_V1_1.00u
- M40: value SWITCH-SPST-2TV -> '
- M41: value SWITCH-SPST-2TV -> Enter; footprint Kailh_Pog:SW_Kailh_Choc_V1_1.00u -> Kailh_Pog:SW_Kailh_Choc_V1_2.25u
- M42: value SWITCH-SPST-2TV -> LeftShift; footprint Kailh_Pog:SW_Kailh_Choc_V1_1.00u -> Kailh_Pog:SW_Kailh_Choc_V1_2.25u
- M43: value SWITCH-SPST-2TV -> Z
- M44: value SWITCH-SPST-2TV -> X
- M45: value SWITCH-SPST-2TV -> C
- M46: value SWITCH-SPST-2TV -> V
- M47: value SWITCH-SPST-2TV -> B
- M48: value SWITCH-SPST-2TV -> N
- M49: value SWITCH-SPST-2TV -> M
- M5: value SWITCH-SPST-2TV -> 4; footprint Kailh_Pog:SW_Kailh_Choc_V1_2.25u -> Kailh_Pog:SW_Kailh_Choc_V1_1.00u
- M50: value SWITCH-SPST-2TV -> ,
- M51: value SWITCH-SPST-2TV -> .
- M52: value SWITCH-SPST-2TV -> /
- M53: value SWITCH-SPST-2TV -> RightShift; footprint Kailh_Pog:SW_Kailh_Choc_V1_1.00u -> Kailh_Pog:SW_Kailh_Choc_V1_2.75u
- M54: value SWITCH-SPST-2TV -> LeftCtrl; footprint Kailh_Pog:SW_Kailh_Choc_V1_1.00u -> Kailh_Pog:SW_Kailh_Choc_V1_1.25u
- M55: value SWITCH-SPST-2TV -> LeftSuper; footprint Kailh_Pog:SW_Kailh_Choc_V1_1.00u -> Kailh_Pog:SW_Kailh_Choc_V1_1.25u
- M56: value SWITCH-SPST-2TV -> LeftAlt; footprint Kailh_Pog:SW_Kailh_Choc_V1_1.00u -> Kailh_Pog:SW_Kailh_Choc_V1_1.25u
- M57: value SWITCH-SPST-2TV -> SpaceBar; footprint Kailh_Pog:SW_Kailh_Choc_V1_1.00u -> Kailh_Pog:SW_Kailh_Choc_V1_6.25u
- M58: value SWITCH-SPST-2TV -> RightAlt; footprint Kailh_Pog:SW_Kailh_Choc_V1_1.00u -> Kailh_Pog:SW_Kailh_Choc_V1_1.25u
- M59: value SWITCH-SPST-2TV -> RightSuper; footprint Kailh_Pog:SW_Kailh_Choc_V1_1.00u -> Kailh_Pog:SW_Kailh_Choc_V1_1.25u
- M6: value SWITCH-SPST-2TV -> 5; footprint Kailh_Pog:SW_Kailh_Choc_V1_2.25u -> Kailh_Pog:SW_Kailh_Choc_V1_1.00u
- M60: value SWITCH-SPST-2TV -> Menu; footprint Kailh_Pog:SW_Kailh_Choc_V1_1.00u -> Kailh_Pog:SW_Kailh_Choc_V1_1.25u
- M61: value SWITCH-SPST-2TV -> RightCtrl; footprint Kailh_Pog:SW_Kailh_Choc_V1_1.00u -> Kailh_Pog:SW_Kailh_Choc_V1_1.25u
- M7: value SWITCH-SPST-2TV -> 6; footprint Kailh_Pog:SW_Kailh_Choc_V1_2.75u -> Kailh_Pog:SW_Kailh_Choc_V1_1.00u
- M8: value SWITCH-SPST-2TV -> 7; footprint Kailh_Pog:SW_Kailh_Choc_V1_1.25u -> Kailh_Pog:SW_Kailh_Choc_V1_1.00u
- M9: value SWITCH-SPST-2TV -> 8; footprint Kailh_Pog:SW_Kailh_Choc_V1_1.25u -> Kailh_Pog:SW_Kailh_Choc_V1_1.00u
- R1, R2: value R_Small -> 10k; moved to F.Cu
- U1: value PCF8575TS_1,118 -> ROW_1_2; footprint NXP:NXP-SOT340-1-02_2016-0-MFG -> MCP23017:SOIC127P1030X265-28N; moved to F.Cu
- U2: value PCF8575TS_1,118 -> ROW_3_4; footprint NXP:NXP-SOT340-1-02_2016-0-MFG -> MCP23017:SOIC127P1030X265-28N; moved to F.Cu
- U3: value SeeeduinoXIAO -> ROW_5_6; footprint RP2040:Seeeduino XIAO-MOUDLE14P-2.54-21X17.8MM -> MCP23017:SOIC127P1030X265-28N; moved to F.Cu
- U4: value PCF8575TS_1,118 -> ROW_7_8; footprint NXP:NXP-SOT340-1-02_2016-0-MFG -> MCP23017:SOIC127P1030X265-28N; moved to F.Cu
- moved M1 266.4 mm to (14.3, 57.1)
- moved M3 232.7 mm to (52.4, 57.1)
- moved U1 232.2 mm to (85.7, 132.6), turned to 90 degrees
- moved M29 228.9 mm to (21.4, 95.2)
- moved M16 187.6 mm to (42.9, 76.2)
- moved M5 187.5 mm to (90.5, 57.1)
- moved M32 182.3 mm to (85.7, 95.2)
- moved M11 173.8 mm to (204.8, 57.1)
- moved U4 168.7 mm to (185.7, 133.3), turned to 90 degrees
- moved M26 167.8 mm to (233.4, 76.2)
- moved M54 162.5 mm to (16.7, 133.3)
- moved M46 161.3 mm to (114.3, 114.3)
- moved M27 159.7 mm to (252.4, 76.2)
- moved M55 158.2 mm to (40.5, 133.3)
- moved U3 151.9 mm to (164.3, 133.3), turned to 90 degrees
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Connections:
- M1 pad 2: +5V -> GND
- M10 pad 2: +5V -> GND
- M11 pad 1: /ROW_3_1 -> /ROW_2_2
- M11 pad 2: +5V -> GND
- M12 pad 1: /ROW_4_1 -> /ROW_2_3
- M12 pad 2: +5V -> GND
- M13 pad 1: /ROW_5_1 -> /ROW_2_4
- M13 pad 2: +5V -> GND
- M14 pad 1: /ROW_6_1 -> /ROW_2_5
- M14 pad 2: +5V -> GND
- M15 pad 1: /ROW_7_1 -> /ROW_2_6
- M15 pad 2: +5V -> GND
- M16 pad 1: /ROW_8_1 -> /ROW_2_7
- M16 pad 2: +5V -> GND
- M17 pad 1: /ROW_1_2 -> /ROW_3_0
- M17 pad 2: +5V -> GND
- M18 pad 1: /ROW_2_2 -> /ROW_3_1
- M18 pad 2: +5V -> GND
- M19 pad 2: +5V -> GND
- M2 pad 1: /ROW_2_0 -> /ROW_1_1
- M2 pad 2: +5V -> GND
- M20 pad 1: /ROW_4_2 -> /ROW_3_3
- M20 pad 2: +5V -> GND
- M21 pad 1: /ROW_5_2 -> /ROW_3_4
- M21 pad 2: +5V -> GND
- M22 pad 1: /ROW_6_2 -> /ROW_3_5
- M22 pad 2: +5V -> GND
- M23 pad 1: /ROW_7_2 -> /ROW_3_6
- M23 pad 2: +5V -> GND
- M24 pad 1: /ROW_8_2 -> /ROW_3_7
- M24 pad 2: +5V -> GND
- M25 pad 1: /ROW_1_3 -> /ROW_4_0
- M25 pad 2: +5V -> GND
- M26 pad 1: /ROW_2_3 -> /ROW_4_1
- M26 pad 2: +5V -> GND
- M27 pad 1: /ROW_3_3 -> /ROW_4_2
- M27 pad 2: +5V -> GND
- M28 pad 2: +5V -> GND
- M29 pad 1: /ROW_5_3 -> /ROW_4_4
- M29 pad 2: +5V -> GND
- M3 pad 1: /ROW_3_0 -> /ROW_1_2
- M3 pad 2: +5V -> GND
- M30 pad 1: /ROW_6_3 -> /ROW_4_5
- M30 pad 2: +5V -> GND
- M31 pad 1: /ROW_7_3 -> /ROW_4_6
- M31 pad 2: +5V -> GND
- M32 pad 1: /ROW_8_3 -> /ROW_4_7
- M32 pad 2: +5V -> GND
- M33 pad 1: /ROW_1_4 -> /ROW_5_0
- M33 pad 2: +5V -> GND
- M34 pad 1: /ROW_2_4 -> /ROW_5_1
- M34 pad 2: +5V -> GND
- M35 pad 1: /ROW_3_4 -> /ROW_5_2
- M35 pad 2: +5V -> GND
- M36 pad 1: /ROW_4_4 -> /ROW_5_3
- M36 pad 2: +5V -> GND
- M37 pad 2: +5V -> GND
- M38 pad 1: /ROW_6_4 -> /ROW_5_5
- M38 pad 2: +5V -> GND
- M39 pad 1: /ROW_7_4 -> /ROW_5_6
- M39 pad 2: +5V -> GND
- M4 pad 1: /ROW_4_0 -> /ROW_1_3
- M4 pad 2: +5V -> GND
- M40 pad 1: /ROW_8_4 -> /ROW_5_7
- M40 pad 2: +5V -> GND
- M41 pad 1: /ROW_1_5 -> /ROW_6_0
- M41 pad 2: +5V -> GND
- M42 pad 1: /ROW_2_5 -> /ROW_6_1
- M42 pad 2: +5V -> GND
- M43 pad 1: /ROW_3_5 -> /ROW_6_2
- M43 pad 2: +5V -> GND
- M44 pad 1: /ROW_4_5 -> /ROW_6_3
- M44 pad 2: +5V -> GND
- M45 pad 1: /ROW_5_5 -> /ROW_6_4
- M45 pad 2: +5V -> GND
- M46 pad 2: +5V -> GND
- M47 pad 1: /ROW_7_5 -> /ROW_6_6
- M47 pad 2: +5V -> GND
- M48 pad 1: /ROW_1_6 -> /ROW_6_7
- M48 pad 2: +5V -> GND
- M49 pad 1: /ROW_2_6 -> /ROW_7_0
- M49 pad 2: +5V -> GND
- M5 pad 1: /ROW_5_0 -> /ROW_1_4
- M5 pad 2: +5V -> GND
- M50 pad 1: /ROW_3_6 -> /ROW_7_1
- M50 pad 2: +5V -> GND
- M51 pad 1: /ROW_4_6 -> /ROW_7_2
- M51 pad 2: +5V -> GND
- M52 pad 1: /ROW_5_6 -> /ROW_7_3
- M52 pad 2: +5V -> GND
- M53 pad 1: /ROW_6_6 -> /ROW_7_4
- M53 pad 2: +5V -> GND
- M54 pad 1: /ROW_7_6 -> /ROW_7_5
- M54 pad 2: +5V -> GND
- M55 pad 1: /ROW_1_7 -> /ROW_7_6
- M55 pad 2: +5V -> GND
- M56 pad 1: /ROW_2_7 -> /ROW_7_7
- M56 pad 2: +5V -> GND
- M57 pad 1: /ROW_3_7 -> /ROW_8_0
- M57 pad 2: +5V -> GND
- M58 pad 1: /ROW_4_7 -> /ROW_8_1
- M58 pad 2: +5V -> GND
- M59 pad 1: /ROW_5_7 -> /ROW_8_2
- M59 pad 2: +5V -> GND
- M6 pad 1: /ROW_6_0 -> /ROW_1_5
- M6 pad 2: +5V -> GND
- M60 pad 1: /ROW_6_7 -> /ROW_8_3
- M60 pad 2: +5V -> GND
- M61 pad 1: /ROW_7_7 -> /ROW_8_4
- M61 pad 2: +5V -> GND
- M7 pad 1: /ROW_7_0 -> /ROW_1_6
- M7 pad 2: +5V -> GND
- M8 pad 1: /ROW_8_0 -> /ROW_1_7
- M8 pad 2: +5V -> GND
- M9 pad 1: /ROW_1_1 -> /ROW_2_0
- M9 pad 2: +5V -> GND
- U1 pad 1: /INT_0x0 -> /ROW_2_0
- U1 pad 10: /ROW_1_6 -> GND
- U1 pad 11: /ROW_1_7 -> (no net)
- U1 pad 12: GND -> /SCL_
- U1 pad 13: /ROW_2_0 -> /SDA_
- U1 pad 14: /ROW_2_1 -> (no net)
- U1 pad 15: /ROW_2_2 -> GND
- U1 pad 16: /ROW_2_3 -> GND
- U1 pad 17: /ROW_2_4 -> GND
- U1 pad 18: /ROW_2_5 -> (no net)
- U1 pad 19: /ROW_2_6 -> /INT_0x0
- U1 pad 2: GND -> /ROW_2_1
- U1 pad 20: /ROW_2_7 -> /INT_0x0
- U1 pad 21: GND -> /ROW_1_0
- U1 pad 22: /SCL_ -> /ROW_1_1
- U1 pad 23: /SDA_ -> /ROW_1_2
- U1 pad 24: +5V -> /ROW_1_3
- U1 pad 3: GND -> /ROW_2_2
- U1 pad 4: /ROW_1_0 -> /ROW_2_3
- U1 pad 5: /ROW_1_1 -> /ROW_2_4
- U1 pad 6: /ROW_1_2 -> /ROW_2_5
- U1 pad 7: /ROW_1_3 -> /ROW_2_6
- U1 pad 8: /ROW_1_4 -> /ROW_2_7
- U1 pad 9: /ROW_1_5 -> +5V
- U2 pad 1: /INT_0x2 -> /ROW_4_0
- U2 pad 10: /ROW_5_6 -> GND
- U2 pad 11: /ROW_5_7 -> (no net)
- U2 pad 12: GND -> /SCL_
- U2 pad 13: /ROW_6_0 -> /SDA_
- U2 pad 14: /ROW_6_1 -> (no net)
- U2 pad 15: /ROW_6_2 -> +5V
- U2 pad 16: /ROW_6_3 -> GND
- U2 pad 17: /ROW_6_4 -> GND
- U2 pad 18: /ROW_6_5 -> (no net)
- U2 pad 19: /ROW_6_6 -> /INT_0x1
- U2 pad 2: +5V -> /ROW_4_1
- U2 pad 20: /ROW_6_7 -> /INT_0x1
- U2 pad 21: GND -> /ROW_3_0
- U2 pad 22: /SCL_ -> /ROW_3_1
- U2 pad 23: /SDA_ -> /ROW_3_2
- U2 pad 24: +5V -> /ROW_3_3
- U2 pad 3: GND -> /ROW_4_2
- U2 pad 4: /ROW_5_0 -> /ROW_4_3
- U2 pad 5: /ROW_5_1 -> /ROW_4_4
- U2 pad 6: /ROW_5_2 -> /ROW_4_5
- U2 pad 7: /ROW_5_3 -> /ROW_4_6
- U2 pad 8: /ROW_5_4 -> /ROW_4_7
- U2 pad 9: /ROW_5_5 -> +5V
- U3 pad 1: /INT_0x0 -> /ROW_6_0
- U3 pad 10: (no net) -> GND
- U3 pad 12: (no net) -> /SCL_
- U3 pad 13: GND -> /SDA_
- U3 pad 14: +5V -> (no net)
- U3 pad 15: (no net) -> GND
- U3 pad 16: (no net) -> +5V
- U3 pad 17: (no net) -> GND
- U3 pad 19: (no net) -> /INT_0x2
- U3 pad 2: /INT_0x1 -> /ROW_6_1
- U3 pad 20: (no net) -> /INT_0x2
- U3 pad 3: /INT_0x2 -> /ROW_6_2
- U3 pad 4: /INT_0x3 -> /ROW_6_3
- U3 pad 5: /SDA_ -> /ROW_6_4
- U3 pad 6: /SCL_ -> /ROW_6_5
- U3 pad 7: (no net) -> /ROW_6_6
- U3 pad 8: (no net) -> /ROW_6_7
- U3 pad 9: (no net) -> +5V
- U4 pad 1: /INT_0x1 -> /ROW_8_0
- U4 pad 10: /ROW_3_6 -> GND
- U4 pad 11: /ROW_3_7 -> (no net)
- U4 pad 12: GND -> /SCL_
- U4 pad 13: /ROW_4_0 -> /SDA_
- U4 pad 14: /ROW_4_1 -> (no net)
- U4 pad 15: /ROW_4_2 -> +5V
- U4 pad 16: /ROW_4_3 -> +5V
- U4 pad 17: /ROW_4_4 -> GND
- U4 pad 18: /ROW_4_5 -> (no net)
- U4 pad 19: /ROW_4_6 -> /INT_0x3
- U4 pad 2: GND -> /ROW_8_1
- U4 pad 20: /ROW_4_7 -> /INT_0x3
- U4 pad 21: +5V -> /ROW_7_0
- U4 pad 22: /SCL_ -> /ROW_7_1
- U4 pad 23: /SDA_ -> /ROW_7_2
- U4 pad 24: +5V -> /ROW_7_3
- U4 pad 3: GND -> /ROW_8_2
- U4 pad 4: /ROW_3_0 -> /ROW_8_3
- U4 pad 5: /ROW_3_1 -> /ROW_8_4
- U4 pad 6: /ROW_3_2 -> (no net)
- U4 pad 7: /ROW_3_3 -> (no net)
- U4 pad 8: /ROW_3_4 -> (no net)
- U4 pad 9: /ROW_3_5 -> +5V
Routing:
- net +5V: track 1369.2 -> 0.00 mm
- net /SDA_: track 0.00 -> 3.02 mm
- net /SCL_: track 0.00 -> 3.02 mm
- net /ROW_1_4: track 2.75 -> 0.00 mm
- net /ROW_6_0: track 2.74 -> 0.00 mm
- net /ROW_4_4: track 2.74 -> 0.00 mm
- net /ROW_6_1: track 2.74 -> 0.00 mm
