File: keyboard.sch (KiCad schematic (older format))
At the start: 68 parts, among them M1 `, M10 9, M11 0, M12 -, M13 =, M14 Backspace, M15 Tab, M16 Q, M17 W, M18 E, M19 R, M2 1, M20 T, M21 Y, M22 U, M23 I, M24 O, M25 P, M26 [, M27 ], M28 \\, M29 CapsLock, M3 2, M30 A, M31 S, M32 D, M33 F, M34 G, M35 H, M36 J, M37 K, M38 L, M39 ;, M4 3, M40 ', M41 Enter, M42 LeftShift, M43 Z, M44 X, M45 C, M46 V, M47 B, M48 N, M49 M, M5 4, M50 ,, M51 ., M52 /, M53 RightShift, M54 LeftCtrl, M55 LeftSuper, M56 LeftAlt, M57 SpaceBar, M58 RightAlt, M59 RightSuper, M6 5, M60 Menu, M61 RightCtrl, M7 6, M8 7, M9 8, U1 ROW_1_2, U2 ROW_3_4, U3 ROW_5_6, U3 SeeeduinoXIAO, U4 ROW_7_8

Commit message: routing
Parts:
- C1: renamed from U3; symbol RP2040:SeeeduinoXIAO -> keyboard-rescue:SeeeduinoXIAO-RP2040
- M1, M10, M11, M12, M13, M14, M15, M16, M17, M18, M19, M2, M20, M21, M22, M23, M24, M25, M26, M27, M28, M29, M3, M30, M31, M32, M33, M34, M35, M36, M37, M38, M39, M4, M40, M41, M42, M43, M44, M45, M46, M47, M48, M49, M5, M50, M51, M52, M53, M54, M55, M56, M57, M58, M59, M6, M60, M61, M7, M8, M9: symbol SparkFun-Electromechanical:SWITCH-SPST-2TV -> keyboard-rescue:SWITCH-SPST-2TV-SparkFun-Electromechanical
- U1, U2, U3, U4: symbol MCP23017:MCP23017T-E_SO -> keyboard-rescue:MCP23017T-E_SO-MCP23017
Connections:
- no-connect marks 15 -> 19

Commit message: Prototype 1
Parts:
- removed M48: N, Kailh_Pog:SW_Kailh_Choc_V1_1.00u, symbol keyboard-rescue:SWITCH-SPST-2TV-SparkFun-Electromechanical
- removed M49: M, Kailh_Pog:SW_Kailh_Choc_V1_1.00u, symbol keyboard-rescue:SWITCH-SPST-2TV-SparkFun-Electromechanical
- removed M50: ,, Kailh_Pog:SW_Kailh_Choc_V1_1.00u, symbol keyboard-rescue:SWITCH-SPST-2TV-SparkFun-Electromechanical
- removed M51: ., Kailh_Pog:SW_Kailh_Choc_V1_1.00u, symbol keyboard-rescue:SWITCH-SPST-2TV-SparkFun-Electromechanical
- removed M52: /, Kailh_Pog:SW_Kailh_Choc_V1_1.00u, symbol keyboard-rescue:SWITCH-SPST-2TV-SparkFun-Electromechanical
- removed M53: RightShift, Kailh_Pog:SW_Kailh_Choc_V1_2.75u, symbol keyboard-rescue:SWITCH-SPST-2TV-SparkFun-Electromechanical
- removed M54: LeftCtrl, Kailh_Pog:SW_Kailh_Choc_V1_1.25u, symbol keyboard-rescue:SWITCH-SPST-2TV-SparkFun-Electromechanical
- removed M55: LeftSuper, Kailh_Pog:SW_Kailh_Choc_V1_1.25u, symbol keyboard-rescue:SWITCH-SPST-2TV-SparkFun-Electromechanical
- removed M56: LeftAlt, Kailh_Pog:SW_Kailh_Choc_V1_1.25u, symbol keyboard-rescue:SWITCH-SPST-2TV-SparkFun-Electromechanical
- removed M57: SpaceBar, Kailh_Pog:SW_Kailh_Choc_V1_6.25u, symbol keyboard-rescue:SWITCH-SPST-2TV-SparkFun-Electromechanical
- removed M58: RightAlt, Kailh_Pog:SW_Kailh_Choc_V1_1.25u, symbol keyboard-rescue:SWITCH-SPST-2TV-SparkFun-Electromechanical
- removed M59: RightSuper, Kailh_Pog:SW_Kailh_Choc_V1_1.25u, symbol keyboard-rescue:SWITCH-SPST-2TV-SparkFun-Electromechanical
- removed M60: Menu, Kailh_Pog:SW_Kailh_Choc_V1_1.25u, symbol keyboard-rescue:SWITCH-SPST-2TV-SparkFun-Electromechanical
- removed M61: RightCtrl, Kailh_Pog:SW_Kailh_Choc_V1_1.25u, symbol keyboard-rescue:SWITCH-SPST-2TV-SparkFun-Electromechanical
- added H1, H2, H3, H4: MountingHole, MountingHole:MountingHole_3.2mm_M3_Pad, symbol Mechanical:MountingHole
- M1: value ` -> Tab
- M10: value 9 -> O
- M11: value 0 -> P
- M12: value - -> Backspace
- M13: value = -> Esc
- M14: value Backspace -> A; footprint Kailh_Pog:SW_Kailh_Choc_V1_2.00u -> Kailh_Pog:SW_Kailh_Choc_V1_1.00u
- M15: value Tab -> S; footprint Kailh_Pog:SW_Kailh_Choc_V1_1.50u -> Kailh_Pog:SW_Kailh_Choc_V1_1.00u
- M16: value Q -> D
- M17: value W -> F
- M18: value E -> G
- M19: value R -> H
- M2: value 1 -> Q
- M20: value T -> J
- M21: value Y -> K
- M22: value U -> L
- M23: value I -> ;
- M24: value O -> '
- M25: value P -> Shift
- M26: value [ -> Z
- M27: value ] -> X
- M28: value \\ -> C; footprint Kailh_Pog:SW_Kailh_Choc_V1_1.50u -> Kailh_Pog:SW_Kailh_Choc_V1_1.00u
- M29: value CapsLock -> V; footprint Kailh_Pog:SW_Kailh_Choc_V1_1.75u -> Kailh_Pog:SW_Kailh_Choc_V1_1.00u
- M3: value 2 -> W
- M30: value A -> B
- M31: value S -> N
- M32: value D -> M
- M33: value F -> ,
- M34: value G -> .
- M35: value H -> /
- M36: value J -> Enter
- M37: value K -> Blnk
- M38: value L -> Ctrl
- M39: value ; -> Alt
- M4: value 3 -> E
- M40: value ' -> Super
- M41: value Enter -> Down; footprint Kailh_Pog:SW_Kailh_Choc_V1_2.25u -> Kailh_Pog:SW_Kailh_Choc_V1_1.00u
- M42: value LeftShift -> Space; footprint Kailh_Pog:SW_Kailh_Choc_V1_2.25u -> Kailh_Pog:SW_Kailh_Choc_V1_2.00u
- M43: value Z -> Up
- M44: value X -> L_Ar
- M45: value C -> D_Ar
- M46: value V -> U_Ar
- M47: value B -> R_Ar
- M5: value 4 -> R
- M6: value 5 -> T
- M7: value 6 -> Y
- M8: value 7 -> U
- M9: value 8 -> I
- U1: value ROW_1_2 -> ROW_1
- U2: value ROW_3_4 -> ROW_2
- U3: value ROW_5_6 -> ROW_3
- U4: value ROW_7_8 -> ROW_4
Connections:
- net ROW_7_3 is gone; now on net ROW_4_7: U4.24 (GPA3)
- net ROW_7_4 is gone; now on net ROW_4_6: U4.25 (GPA4)
- net ROW_7_5 is gone; now on net ROW_4_5: U4.26 (GPA5)
- net ROW_7_6 is gone; now on net ROW_4_4: U4.27 (GPA6)
- net ROW_7_7 is gone; now on net ROW_4_3: U4.28 (GPA7)
- net ROW_8_0 is gone; now on net ROW_4_0: U4.1 (GPB0)
- net ROW_8_1 is gone; now on net ROW_4_1: U4.2 (GPB1)
- net ROW_8_2 is gone; now on net ROW_4_2: U4.3 (GPB2)
- net +5V: now also U1.18 (~RESET), U2.18 (~RESET), U3.18 (~RESET), U4.18 (~RESET)
- net ROW_1_0: now also U1.1 (GPB0); no longer U1.28 (GPA7)
- net ROW_1_1: now also U1.2 (GPB1); no longer U1.27 (GPA6)
- net ROW_1_2: now also U1.3 (GPB2); no longer U1.26 (GPA5)
- net ROW_1_3: now also U1.4 (GPB3); no longer U1.25 (GPA4)
- net ROW_1_4: now also U1.28 (GPA7); no longer U1.24 (GPA3)
- net ROW_1_5: now also U1.27 (GPA6); no longer U1.23 (GPA2)
- net ROW_1_6: now also U1.26 (GPA5); no longer U1.22 (GPA1)
- net ROW_1_7: now also U1.25 (GPA4); no longer U1.21 (GPA0)
- net ROW_2_0: now also M13.1 (O), U2.1 (GPB0); no longer M9.1 (O), U1.1 (GPB0)
- net ROW_2_1: now also M14.1 (O), U2.2 (GPB1); no longer M10.1 (O), U1.2 (GPB1)
- net ROW_2_2: now also M15.1 (O), U2.3 (GPB2); no longer M11.1 (O), U1.3 (GPB2)
- net ROW_2_3: now also M16.1 (O), U2.4 (GPB3); no longer M12.1 (O), U1.4 (GPB3)
- net ROW_2_4: now also M17.1 (O), U2.28 (GPA7); no longer M13.1 (O), U1.5 (GPB4)
- net ROW_2_5: now also M18.1 (O), U2.27 (GPA6); no longer M14.1 (O), U1.6 (GPB5)
- net ROW_2_6: now also M19.1 (O), U2.26 (GPA5); no longer M15.1 (O), U1.7 (GPB6)
- net ROW_2_7: now also M20.1 (O), U2.25 (GPA4); no longer M16.1 (O), U1.8 (GPB7)
- net ROW_3_0: now also M25.1 (O), U3.1 (GPB0); no longer M17.1 (O), U2.21 (GPA0)
- net ROW_3_1: now also M26.1 (O), U3.2 (GPB1); no longer M18.1 (O), U2.22 (GPA1)
- net ROW_3_2: now also M27.1 (O), U3.3 (GPB2); no longer M19.1 (O), U2.23 (GPA2)
- net ROW_3_3: now also M28.1 (O), U3.4 (GPB3); no longer M20.1 (O), U2.24 (GPA3)
- net ROW_3_4: now also M29.1 (O), U3.28 (GPA7); no longer M21.1 (O), U2.25 (GPA4)
- net ROW_3_5: now also M30.1 (O), U3.27 (GPA6); no longer M22.1 (O), U2.26 (GPA5)
- net ROW_3_6: now also M31.1 (O), U3.26 (GPA5); no longer M23.1 (O), U2.27 (GPA6)
- net ROW_3_7: now also M32.1 (O), U3.25 (GPA4); no longer M24.1 (O), U2.28 (GPA7)
- net ROW_4_0: now also M37.1 (O); no longer M25.1 (O), U2.1 (GPB0)
- net ROW_4_1: now also M38.1 (O); no longer M26.1 (O), U2.2 (GPB1)
- net ROW_4_2: now also M39.1 (O); no longer M27.1 (O), U2.3 (GPB2)
- net ROW_4_3: now also M40.1 (O); no longer M28.1 (O), U2.4 (GPB3)
- net ROW_4_4: now also M41.1 (O); no longer M29.1 (O), U2.5 (GPB4)
- net ROW_4_5: now also M42.1 (O); no longer M30.1 (O), U2.6 (GPB5)
- net ROW_4_6: now also M43.1 (O); no longer M31.1 (O), U2.7 (GPB6)
- net ROW_4_7: now also M44.1 (O); no longer M32.1 (O), U2.8 (GPB7)
- net INT_0x4: now reaches C1.7 (PB08_A6_D6_TX)
- net ROW_5_0 renamed ROW_3_11
- net ROW_3_11: now also M36.1 (O); no longer M33.1 (O)
- net ROW_5_1 renamed ROW_3_10
- net ROW_3_10: now also M35.1 (O); no longer M34.1 (O)
- net ROW_5_2 renamed ROW_3_9
- net ROW_3_9: now also M34.1 (O); no longer M35.1 (O)
- net ROW_5_3 renamed ROW_3_8
- net ROW_3_8: now also M33.1 (O); no longer M36.1 (O)
- removed net ROW_5_4: M37.1 (O), U3.25 (GPA4)
- removed net ROW_5_5: M38.1 (O), U3.26 (GPA5)
- removed net ROW_5_6: M39.1 (O), U3.27 (GPA6)
- removed net ROW_5_7: M40.1 (O), U3.28 (GPA7)
- removed net ROW_6_0: M41.1 (O), U3.1 (GPB0)
- removed net ROW_6_1: M42.1 (O), U3.2 (GPB1)
- removed net ROW_6_2: M43.1 (O), U3.3 (GPB2)
- removed net ROW_6_3: M44.1 (O), U3.4 (GPB3)
- net ROW_6_4: no longer names the net of U3.5 (GPB4)
- net ROW_6_4: no longer M45.1 (O)
- net ROW_6_5: no longer names the net of U3.6 (GPB5)
- net ROW_6_5: no longer M46.1 (O)
- net ROW_6_6: no longer names the net of U3.7 (GPB6)
- net ROW_6_6: no longer M47.1 (O)
- net ROW_6_7: no longer names the net of U3.8 (GPB7)
- net ROW_7_0 renamed ROW_4_10
- net ROW_4_10: now also M47.1 (O)
- net ROW_7_1 renamed ROW_4_9
- net ROW_4_9: now also M46.1 (O)
- net ROW_7_2 renamed ROW_4_8
- net ROW_4_8: now also M45.1 (O)
- net ROW_8_3: no longer names the net of U4.4 (GPB3)
- net ROW_8_4: no longer names the net of U4.5 (GPB4)
- new net ROW_1_10: M11.1 (O), U1.22 (GPA1)
- new net ROW_1_11: M12.1 (O), U1.21 (GPA0)
- new net ROW_1_8: M9.1 (O), U1.24 (GPA3)
- new net ROW_1_9: M10.1 (O), U1.23 (GPA2)
- new net ROW_2_10: M23.1 (O), U2.22 (GPA1)
- new net ROW_2_11: M24.1 (O), U2.21 (GPA0)
- new net ROW_2_8: M21.1 (O), U2.24 (GPA3)
- new net ROW_2_9: M22.1 (O), U2.23 (GPA2)
- no-connect marks 19 -> 32
Other:
- moved on the sheet: M1, M10, M11, M12, M13, M14, M15, M16, M17, M18, M19, M2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
