File: Hardware/keyboard.kicad_pcb (KiCad board)
At the start: 2 copper layers, 270 x 100 mm, 60 parts, among them M1 Tab, M10 O, M11 P, M12 Backspace, M13 Esc, M14 A, M15 S, M16 D, M17 F, M18 G, M19 H, M2 Q, M20 J, M21 K, M22 L, M23 ;, M24 ', M25 Shift, M26 Z, M27 X, M28 C, M29 V, M3 W, M30 B, M31 N, M32 M, M33 ,, M34 ., M35 /, M36 Enter, M37 Blnk, M38 Ctrl, M39 Alt, M4 E, M40 Super, M41 Down, M42 Space, M43 Up, M44 L_Ar, M45 D_Ar, M46 U_Ar, M47 R_Ar, M5 R, M6 T, M7 Y, M8 U, M9 I, U1 ROW_1, U2 ROW_2, U3 ROW_3, U4 ROW_4

Commit message: South-facing switch change
Parts:
- C1: value Pi Pico -> SeeeduinoXIAO
- M42: footprint Kailh_Pog:SW_Kailh_Choc_V1_2.00u -> Hardware:SW_Kailh_Choc_V1_2.00u
- moved H6 138.9 mm to (327.4, 183.4)
- moved H2 134.9 mm to (199.6, 90.7)
- moved H1 102.4 mm to (327.4, 90.7)
- moved H4 35.9 mm to (70.6, 90.7)
- moved R1 10.3 mm to (75.9, 170.8)
- moved U4 10.3 mm to (86.6, 176.2)
- moved C1 10.3 mm to (78.0, 109.0)
- moved U1 10.3 mm to (86.6, 119.0)
- moved R2 10.3 mm to (75.2, 174.1)
- moved U2 10.3 mm to (86.6, 138.1)
- moved U3 10.3 mm to (86.6, 157.1)
- moved H5 9.70 mm to (199.6, 183.4)
- moved H3 9.63 mm to (70.6, 183.4)
Connections:
- U1 pad 1: /ROW_1_0 -> /ROW_1_3
- U1 pad 2: /ROW_1_1 -> /ROW_1_2
- U1 pad 21: /ROW_1_11 -> /ROW_1_4
- U1 pad 22: /ROW_1_10 -> /ROW_1_5
- U1 pad 23: /ROW_1_9 -> /ROW_1_6
- U1 pad 24: /ROW_1_8 -> /ROW_1_7
- U1 pad 25: /ROW_1_7 -> /ROW_1_8
- U1 pad 26: /ROW_1_6 -> /ROW_1_9
- U1 pad 27: /ROW_1_5 -> /ROW_1_10
- U1 pad 28: /ROW_1_4 -> /ROW_1_11
- U1 pad 3: /ROW_1_2 -> /ROW_1_1
- U1 pad 4: /ROW_1_3 -> /ROW_1_0
- U2 pad 1: /ROW_2_0 -> /ROW_2_3
- U2 pad 2: /ROW_2_1 -> /ROW_2_2
- U2 pad 21: /ROW_2_11 -> /ROW_2_4
- U2 pad 22: /ROW_2_10 -> /ROW_2_5
- U2 pad 23: /ROW_2_9 -> /ROW_2_6
- U2 pad 24: /ROW_2_8 -> /ROW_2_7
- U2 pad 25: /ROW_2_7 -> /ROW_2_8
- U2 pad 26: /ROW_2_6 -> /ROW_2_9
- U2 pad 27: /ROW_2_5 -> /ROW_2_10
- U2 pad 28: /ROW_2_4 -> /ROW_2_11
- U2 pad 3: /ROW_2_2 -> /ROW_2_1
- U2 pad 4: /ROW_2_3 -> /ROW_2_0
- U3 pad 1: /ROW_3_0 -> /ROW_3_3
- U3 pad 2: /ROW_3_1 -> /ROW_3_2
- U3 pad 21: /ROW_3_11 -> /ROW_3_4
- U3 pad 22: /ROW_3_10 -> /ROW_3_5
- U3 pad 23: /ROW_3_9 -> /ROW_3_6
- U3 pad 24: /ROW_3_8 -> /ROW_3_7
- U3 pad 25: /ROW_3_7 -> /ROW_3_8
- U3 pad 26: /ROW_3_6 -> /ROW_3_9
- U3 pad 27: /ROW_3_5 -> /ROW_3_10
- U3 pad 28: /ROW_3_4 -> /ROW_3_11
- U3 pad 3: /ROW_3_2 -> /ROW_3_1
- U3 pad 4: /ROW_3_3 -> /ROW_3_0
- U4 pad 1: /ROW_4_0 -> /ROW_4_2
- U4 pad 21: /ROW_4_10 -> /ROW_4_3
- U4 pad 22: /ROW_4_9 -> /ROW_4_4
- U4 pad 23: /ROW_4_8 -> /ROW_4_5
- U4 pad 24: /ROW_4_7 -> /ROW_4_6
- U4 pad 25: /ROW_4_6 -> /ROW_4_7
- U4 pad 26: /ROW_4_5 -> /ROW_4_8
- U4 pad 27: /ROW_4_4 -> /ROW_4_9
- U4 pad 28: /ROW_4_3 -> /ROW_4_10
- U4 pad 3: /ROW_4_2 -> /ROW_4_0
Routing:
- net /ROW_3_0: track 32.3 -> 35.5 mm
- net /ROW_2_0: track 32.3 -> 35.5 mm
- net /ROW_3_1: track 51.2 -> 53.5 mm
- net /ROW_2_1: track 51.2 -> 53.5 mm
- net /ROW_3_3: track 89.0 -> 91.3 mm
- net /ROW_2_3: track 89.0 -> 91.3 mm
- net /ROW_2_8: track 174.9 -> 177.1 mm
- net /ROW_2_9: track 193.8 -> 196.0 mm
- net /ROW_4_0: track 32.3 -> 34.3 mm
- net /ROW_4_2: track 70.1 -> 71.8 mm
- net /ROW_3_11: track 231.6 -> 233.3 mm
- net /ROW_2_10: track 212.7 -> 214.3 mm
- net /ROW_1_0: track 32.3 -> 33.8 mm
- net /ROW_4_3: track 79.7 -> 81.0 mm
- net /ROW_4_4: track 98.6 -> 99.9 mm
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Other:
- board size 270 x 100 mm -> 264 x 100 mm
